File: 4layertest.kicad_pcb (KiCad board)
At the start: 4 copper layers, 63.5 x 38.1 mm, 6 parts

Commit message: more wrk on power planes
Parts:
- moved C4 1.36 mm to (48.3, 99.4)
- moved C3 1.35 mm to (38.2, 83.8)
Routing:
- net GND: track 82.3 -> 22.7 mm
- net -12V: track 45.3 -> 1.02 mm
- net +12V: track 41.3 -> 9.20 mm, vias 0 -> 1
- removed copper zone on B.Cu, net (none)
